File: pcb/motors.kicad_sch (KiCad schematic)
At the start: 16 parts, among them M1 Stepper_Motor_bipolar, M2 Stepper_Motor_bipolar, M3 Stepper_Motor_bipolar, M4 Stepper_Motor_bipolar, M5 Stepper_Motor_bipolar, M6 Stepper_Motor_bipolar, M7 Stepper_Motor_bipolar, M8 Stepper_Motor_bipolar

Commit message: work
Parts:
- A1, A2, A3, A4, A5, A6, A7, A8: Vendor (none) -> Digi-Key
Connections:
- net GND: now also A1.7 (GND), A2.7 (GND), A3.7 (GND), A4.7 (GND), A5.7 (GND), A6.7 (GND), A7.7 (GND), A8.7 (GND)

Commit message: drivers
Parts:
- removed A1, A2, A3, A4, A5, A6, A7, A8: Pololu_Breakout_A4988, Module:Pololu_Breakout-16_15.2x20.3mm, symbol Driver_Motor:Pololu_Breakout_A4988
Connections:
- net Driver 2/1A: now reaches M2.1
- net Driver 2/1B: now reaches M2.2 (-)
- net Driver 2/2A: now reaches M2.3
- net Driver 2/2B: now reaches M2.4
- net Driver 1/1A: now reaches M1.1
- net Driver 1/1B: now reaches M1.2 (-)
- net Driver 1/2A: now reaches M1.3
- net Driver 1/2B: now reaches M1.4
- net Driver 6/1B: now reaches M6.2 (-)
- net Driver 6/1A: now reaches M6.1
- net Driver 6/2A: now reaches M6.3
- net Driver 6/2B: now reaches M6.4
- net Driver 4/1A: now reaches M4.1
- net Driver 4/1B: now reaches M4.2 (-)
- net Driver 4/2A: now reaches M4.3
- net Driver 4/2B: now reaches M4.4
- net Driver 7/1B: now reaches M7.2 (-)
- net Driver 7/1A: now reaches M7.1
- net Driver 7/2A: now reaches M7.3
- net Driver 7/2B: now reaches M7.4
- net Driver 3/1A: now reaches M3.1
- net Driver 3/1B: now reaches M3.2 (-)
- net Driver 3/2A: now reaches M3.3
- net Driver 3/2B: now reaches M3.4
- net Driver 5/1A: now reaches M5.1
- net Driver 5/1B: now reaches M5.2 (-)
- net Driver 5/2A: now reaches M5.3
- net Driver 5/2B: now reaches M5.4
- net Driver 8/1B: now reaches M8.2 (-)
- net Driver 8/1A: now reaches M8.1
- net Driver 8/2A: now reaches M8.3
- net Driver 8/2B: now reaches M8.4
Other:
- added sheet Driver 1 (driver.kicad_sch)
- added sheet Driver 2 (driver.kicad_sch)
- added sheet Driver 3 (driver.kicad_sch)
- added sheet Driver 4 (driver.kicad_sch)
- added sheet Driver 5 (driver.kicad_sch)
- added sheet Driver 6 (driver.kicad_sch)
- added sheet Driver 7 (driver.kicad_sch)
- added sheet Driver 8 (driver.kicad_sch)

Commit message: w
Parts:
- removed M1, M2, M3, M4, M5, M6, M7, M8: Stepper_Motor_bipolar, symbol Motor:Stepper_Motor_bipolar
- added M1, M2, M3, M4, M5, M6, M7, M8: Stepper_Motor_unipolar_6pin, Connector_JST:JST_PH_B6B-PH-K_1x06_P2.00mm_Vertical, symbol Motor:Stepper_Motor_unipolar_6pin
Connections:
- net Driver 1/1A: now also M1.1
- net Driver 1/1B: now also M1.3 (-)
- net Driver 1/2A: now also M1.4
- net Driver 1/2B: now also M1.6
- net Driver 2/1A: now also M2.1
- net Driver 2/1B: now also M2.3 (-)
- net Driver 2/2A: now also M2.4
- net Driver 2/2B: now also M2.6
- net Driver 3/1A: now also M3.1
- net Driver 3/1B: now also M3.3 (-)
- net Driver 3/2A: now also M3.4
- net Driver 3/2B: now also M3.6
- net Driver 4/1A: now also M4.1
- net Driver 4/1B: now also M4.3 (-)
- net Driver 4/2A: now also M4.4
- net Driver 4/2B: now also M4.6
- net Driver 5/1A: now also M5.1
- net Driver 5/1B: now also M5.3 (-)
- net Driver 5/2A: now also M5.4
- net Driver 5/2B: now also M5.6
- net Driver 6/1A: now also M6.1
- net Driver 6/1B: now also M6.3 (-)
- net Driver 6/2A: now also M6.4
- net Driver 6/2B: now also M6.6
- net Driver 7/1A: now also M7.1
- net Driver 7/1B: now also M7.3 (-)
- net Driver 7/2A: now also M7.4
- net Driver 7/2B: now also M7.6
- net Driver 8/1A: now also M8.1
- net Driver 8/1B: now also M8.3 (-)
- net Driver 8/2A: now also M8.4
- net Driver 8/2B: now also M8.6
- no-connect marks 0 -> 16

Commit message: !!!!!
Changed lines of the file:
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@@
 		)
 	)
-	(label "~{ENABLE_3}"
+	(label "ENABLE_3"
 		(at 73.66 168.91 0)
 		(effects
@@
 		)
 	)
-	(label "~{ENABLE_2}"
+	(label "ENABLE_2"
 		(at 73.66 105.41 0)
 		(effects
@@
 		)
 	)
-	(label "~{ENABLE_7}"
+	(label "ENABLE_7"
 		(at 166.37 168.91 0)
 		(effects
@@
 		)
 	)
-	(label "~{ENABLE_6}"
+	(label "ENABLE_6"
 		(at 166.37 105.41 0)
 		(effects
@@
 		)
 	)
-	(label "~{ENABLE_[1..8]}"
+	(label "ENABLE_[1..8]"
 		(at 270.51 86.36 0)
 		(effects
@@
 		)
 	)
-	(label "~{ENABLE_1}"
+	(label "ENABLE_1"
 		(at 73.66 41.91 0)
 		(effects
@@
 		)
 	)
-	(label "~{ENABLE_8}"
+	(label "ENABLE_8"
 		(at 166.37 232.41 0)
 		(effects
@@
 		)
 	)
-	(label "~{ENABLE_4}"
+	(label "ENABLE_4"
 		(at 73.66 232.41 0)
 		(effects
@@
 		)
 	)
-	(label "~{ENABLE_5}"
+	(label "ENABLE_5"
 		(at 166.37 41.91 0)
 		(effects
@@
 		)
 	)
-	(hierarchical_label "~{ENABLE_[1..8]}"
+	(hierarchical_label "ENABLE_[1..8]"
 		(shape output)
 		(at 287.02 86.36 0)
