File: pcb/stepper_music.kicad_pcb (KiCad board)
At the start: 2 copper layers, 56 parts, among them J1 USB_C_Receptacle, J2 Conn_ST_STDC14, J3 MIDI IN, J4 MIDI THRU, U1 STM32F401RCTx, U2 6N138, U3 LD1117S33TR_SOT223, U4 LMR50410, U5 SN74LV1T34DBV, U6 LM66100DCK, U7 LM66100DCK, Y1 25MHz

Commit message: w
Parts:
- added C21: 10μF, Capacitor_SMD:C_1206_3216Metric_Pad1.33x1.80mm_HandSolder, F.Cu at (161.1, 132.9)
- added J5: Conn_01x02, Connector_AMASS:AMASS_XT30PW-M_1x02_P2.50mm_Horizontal, F.Cu at (168.2, 128.5)
- D1: footprint Diode_THT:D_DO-35_SOD27_P7.62mm_Horizontal -> Diode_SMD:D_SOD-523
- L1: footprint Inductor_SMD:L_1206_3216Metric -> Inductor_SMD:L_1008_2520Metric_Pad1.43x2.20mm_HandSolder
- moved A1 115.5 mm to (266.9, 79.0)
- moved A3 115.5 mm to (300.5, 79.0)
- moved A4 115.5 mm to (317.3, 79.0)
- moved A6 115.5 mm to (266.9, 100.8)
- moved A8 115.5 mm to (300.5, 100.8)
- moved A2 115.5 mm to (283.7, 79.0)
- moved A5 115.5 mm to (334.1, 79.0)
- moved A7 115.5 mm to (283.7, 100.8)
- moved U6 112.5 mm to (96.9, 68.6)
- moved U3 111.9 mm to (99.8, 81.0), turned to 180 degrees
- moved J4 111.7 mm to (78.2, 55.5), turned to -90 degrees
- moved U7 111.0 mm to (96.7, 74.5)
- moved C19 103.0 mm to (101.3, 72.3), turned to 180 degrees
- moved U1 102.8 mm to (95.8, 96.8), turned to 180 degrees
- moved C8 99.8 mm to (90.3, 88.9), turned to 90 degrees
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Routing:
- net Net-(U1-PH0): track 0.00 -> 9.14 mm
- net Net-(U1-PH1): track 0.00 -> 9.12 mm
- net GND: vias 0 -> 2
- net +5V: vias 0 -> 2
- net +3.3V: vias 0 -> 2
- added copper zone on B.Cu, net +3.3V
- added copper zone on F.Cu, net +3.3V
- added copper zone on F.Cu, net +5V
- added copper zone on F.Cu, net GND
- added copper zone on In1.Cu, net GND
- added copper zone on In2.Cu, net GND
Other:
- board outline added: 70 x 70 mm
- copper layers 2 -> 4

Commit message: route
Parts:
- moved U2 128.7 mm to (93.6, 72.4)
- moved J5 128.1 mm to (83.9, 32.0), turned to 90 degrees
- moved C21 122.4 mm to (88.2, 34.5), turned to 90 degrees
- moved R10 121.9 mm to (88.5, 52.0), turned to -90 degrees
- moved U5 119.6 mm to (93.0, 58.9)
- moved R9 113.4 mm to (88.5, 62.0), turned to -90 degrees
- moved C18 111.3 mm to (96.4, 59.5), turned to -90 degrees
- moved D1 108.5 mm to (89.2, 72.4), turned to -90 degrees
- moved C11 106.9 mm to (88.3, 77.5), turned to -90 degrees
- moved C17 103.2 mm to (98.6, 72.4), turned to -90 degrees
- moved R5 99.0 mm to (93.6, 67.0), turned to 180 degrees
- moved R6 94.2 mm to (95.7, 76.5), turned to 180 degrees
- moved R4 93.8 mm to (90.3, 83.0)
- moved C16 68.9 mm to (102.7, 66.9), turned to 90 degrees
- moved C14 66.6 mm to (109.5, 66.2), turned to -90 degrees
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Connections:
- net Net-(U6-VIN) renamed /5V_REGOUT
Routing:
- net +5V: track 0.00 -> 32.4 mm, vias 2 -> 0
- net /5V_REGOUT: track 0.00 -> 14.9 mm
- net Net-(D1-K): track 0.00 -> 14.4 mm
- net GND: track 0.00 -> 10.5 mm, vias 2 -> 12
- net Net-(U2-VO1): track 0.00 -> 8.28 mm
- net Net-(U4-FB): track 0.00 -> 8.23 mm
- net Net-(C11-Pad1): track 0.00 -> 6.13 mm
- net Net-(D1-A): track 0.00 -> 5.71 mm
- net /VBUS: track 0.00 -> 5.14 mm
- net /MIDI_RX: track 0.00 -> 4.94 mm
- net +12V: track 0.00 -> 4.74 mm, vias 0 -> 3
- net Net-(J3-Pad4): track 0.00 -> 3.29 mm
- net Net-(J4-Pad4): track 0.00 -> 3.05 mm
- net Net-(U4-CB): track 0.00 -> 2.45 mm
- net +3.3V: vias 2 -> 5
- added copper zone on B.Cu, net +12V
- added copper zone on F.Cu, net +12V
- added copper zone on F.Cu, net /5V_REGOUT
- added copper zone on F.Cu, net Net-(U4-SW)
Other:
- board size 70 x 70 mm -> 70 x 90 mm

Commit message: w
Parts:
- moved TP1 154.2 mm to (46.8, 104.2)
- moved TP4 142.1 mm to (81.6, 63.6)
- moved C20 123.4 mm to (73.5, 116.8), turned to 90 degrees
- moved C10 122.1 mm to (72.4, 134.0)
- moved R1 114.2 mm to (67.5, 129.8)
- moved R2 111.6 mm to (67.5, 116.2)
- moved R3 109.8 mm to (72.4, 137.7)
- moved TP2 107.8 mm to (90.2, 137.1)
- moved C9 102.1 mm to (83.5, 111.8), turned to 90 degrees
- moved TP3 102.1 mm to (105.2, 99.2)
- moved J2 86.4 mm to (81.6, 137.5), turned to 90 degrees
- moved A1 80.2 mm to (186.8, 78.0)
- moved A4 80.2 mm to (237.1, 78.0)
- moved A6 80.2 mm to (186.8, 99.9)
- moved A3 80.2 mm to (220.3, 78.0)
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Routing:
- net /MIDI_RX: track 4.94 -> 29.1 mm
- net GND: track 10.5 -> 31.3 mm, vias 12 -> 26
- net +5V: track 32.4 -> 52.1 mm
- net /~{RST}: track 0.00 -> 16.8 mm
- net /SWDIO: track 0.00 -> 12.7 mm
- net Net-(J1-CC1): track 0.00 -> 10.9 mm
- net /SWCLK: track 0.00 -> 8.74 mm
- net Net-(J1-CC2): track 0.00 -> 8.17 mm
- net Net-(U5-Y): track 0.00 -> 6.34 mm
- net +12V: track 4.74 -> 9.16 mm
- net +3.3V: track 0.00 -> 3.64 mm, vias 5 -> 7
- net Net-(U1-VCAP1): track 0.00 -> 2.93 mm
- net Net-(J4-Pad5): track 0.00 -> 2.62 mm
Other:
- board size 70 x 90 mm -> 70 x 100 mm

Commit message: Update stepper_music.kicad_pcb
Routing:
- net /USB_D+: track 0.00 -> 22.1 mm, vias 0 -> 2
- net /USB_D-: track 0.00 -> 18.9 mm, vias 0 -> 2
- net +5V: track 52.1 -> 51.5 mm
- net GND: vias 26 -> 37

Commit message: drivers
Parts:
- moved A1 74.9 mm to (196.3, 3.71)
- moved A2 51.3 mm to (196.3, 27.3)
- moved A4 40.9 mm to (196.3, 75.3)
- moved A3 36.0 mm to (196.3, 51.3)
- moved TP3 4.14 mm to (106.5, 95.2)
- moved R4 1.57 mm to (79.6, 106.7)
Routing:
- net /VBUS: track 5.14 -> 63.1 mm, vias 0 -> 2
- net /MIDI_RX: track 29.1 -> 57.7 mm
- net /~{RST}: track 16.8 -> 39.1 mm, vias 0 -> 2
- net /SWO: track 0.00 -> 12.1 mm, vias 0 -> 2
- net GND: track 31.3 -> 40.8 mm, vias 37 -> 48
- net /MS3: track 0.00 -> 3.43 mm
- net /MS2: track 0.00 -> 3.36 mm
- net /MS1: track 0.00 -> 3.32 mm
- net /DIR_6: track 0.00 -> 3.28 mm
- net /STEP_2: track 0.00 -> 3.25 mm
- net +3.3V: track 3.64 -> 6.87 mm, vias 7 -> 17
- net /DIR_5: track 0.00 -> 3.21 mm
- net /STEP_3: track 0.00 -> 3.21 mm
- net +5V: track 51.5 -> 52.8 mm
- net Net-(D1-K): track 14.4 -> 13.4 mm
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
Commit message: w
Parts:
- removed A1, A2, A3, A4, A5, A6, A7, A8: Pololu_Breakout_A4988, Module:Pololu_Breakout-16_15.2x20.3mm
- added C22: 220nF, Capacitor_SMD:C_1206_3216Metric_Pad1.33x1.80mm_HandSolder, F.Cu at (114.8, 124.8)
- added C23: 100nF, Capacitor_SMD:C_1206_3216Metric_Pad1.33x1.80mm_HandSolder, F.Cu at (121.2, 122.3)
- added C24: 100nF, Capacitor_SMD:C_1206_3216Metric_Pad1.33x1.80mm_HandSolder, F.Cu at (118.6, 122.3)
- added C25: 220nF, Capacitor_SMD:C_1206_3216Metric_Pad1.33x1.80mm_HandSolder, F.Cu at (117.0, 133.4)
- added C26: 4.7μF, Capacitor_SMD:C_1206_3216Metric_Pad1.33x1.80mm_HandSolder, F.Cu at (121.2, 140.1)
- added C27: 100nF, Capacitor_SMD:C_1206_3216Metric_Pad1.33x1.80mm_HandSolder, F.Cu at (124.5, 132.5)
- added C28: 100nF, Capacitor_SMD:C_1206_3216Metric_Pad1.33x1.80mm_HandSolder, F.Cu at (124.5, 123.5)
- added C29: 100nF, Capacitor_SMD:C_1206_3216Metric_Pad1.33x1.80mm_HandSolder, F.Cu at (203.4, 33.0)
- added C30: 100nF, Capacitor_SMD:C_1206_3216Metric_Pad1.33x1.80mm_HandSolder, F.Cu at (203.4, 36.4)
- added C31: 220nF, Capacitor_SMD:C_1206_3216Metric_Pad1.33x1.80mm_HandSolder, F.Cu at (203.4, 39.8)
- added C32: 220nF, Capacitor_SMD:C_1206_3216Metric_Pad1.33x1.80mm_HandSolder, F.Cu at (203.4, 43.1)
- added C33: 4.7μF, Capacitor_SMD:C_1206_3216Metric_Pad1.33x1.80mm_HandSolder, F.Cu at (203.4, 46.5)
- added C34: 100nF, Capacitor_SMD:C_1206_3216Metric_Pad1.33x1.80mm_HandSolder, F.Cu at (203.4, 49.8)
- added C35: 100nF, Capacitor_SMD:C_1206_3216Metric_Pad1.33x1.80mm_HandSolder, F.Cu at (203.4, 53.1)
- added C36: 100nF, Capacitor_SMD:C_1206_3216Metric_Pad1.33x1.80mm_HandSolder, F.Cu at (227.6, 118.2)
- added C37: 100nF, Capacitor_SMD:C_1206_3216Metric_Pad1.33x1.80mm_HandSolder, F.Cu at (227.6, 121.5)
- added C38: 220nF, Capacitor_SMD:C_1206_3216Metric_Pad1.33x1.80mm_HandSolder, F.Cu at (227.6, 124.9)
- added C39: 220nF, Capacitor_SMD:C_1206_3216Metric_Pad1.33x1.80mm_HandSolder, F.Cu at (227.6, 128.2)
- added C40: 4.7μF, Capacitor_SMD:C_1206_3216Metric_Pad1.33x1.80mm_HandSolder, F.Cu at (227.6, 131.6)
- added C41: 100nF, Capacitor_SMD:C_1206_3216Metric_Pad1.33x1.80mm_HandSolder, F.Cu at (227.6, 134.9)
- added C42: 100nF, Capacitor_SMD:C_1206_3216Metric_Pad1.33x1.80mm_HandSolder, F.Cu at (227.6, 138.3)
- added C43: 100nF, Capacitor_SMD:C_1206_3216Metric_Pad1.33x1.80mm_HandSolder, F.Cu at (206.0, 92.8)
- added C44: 100nF, Capacitor_SMD:C_1206_3216Metric_Pad1.33x1.80mm_HandSolder, F.Cu at (206.0, 96.1)
- added C45: 220nF, Capacitor_SMD:C_1206_3216Metric_Pad1.33x1.80mm_HandSolder, F.Cu at (206.0, 99.5)
- added C46: 220nF, Capacitor_SMD:C_1206_3216Metric_Pad1.33x1.80mm_HandSolder, F.Cu at (206.0, 102.8)
- added C47: 4.7μF, Capacitor_SMD:C_1206_3216Metric_Pad1.33x1.80mm_HandSolder, F.Cu at (206.0, 106.2)
- added C48: 100nF, Capacitor_SMD:C_1206_3216Metric_Pad1.33x1.80mm_HandSolder, F.Cu at (206.0, 109.5)
- added C49: 100nF, Capacitor_SMD:C_1206_3216Metric_Pad1.33x1.80mm_HandSolder, F.Cu at (206.0, 112.8)
- added C50: 100nF, Capacitor_SMD:C_1206_3216Metric_Pad1.33x1.80mm_HandSolder, F.Cu at (206.0, 118.2)
- added C51: 100nF, Capacitor_SMD:C_1206_3216Metric_Pad1.33x1.80mm_HandSolder, F.Cu at (206.0, 121.5)
- added C52: 220nF, Capacitor_SMD:C_1206_3216Metric_Pad1.33x1.80mm_HandSolder, F.Cu at (206.0, 124.9)
- added C53: 220nF, Capacitor_SMD:C_1206_3216Metric_Pad1.33x1.80mm_HandSolder, F.Cu at (206.0, 128.2)
- added C54: 4.7μF, Capacitor_SMD:C_1206_3216Metric_Pad1.33x1.80mm_HandSolder, F.Cu at (206.0, 131.6)
- added C55: 100nF, Capacitor_SMD:C_1206_3216Metric_Pad1.33x1.80mm_HandSolder, F.Cu at (206.0, 134.9)
- added C56: 100nF, Capacitor_SMD:C_1206_3216Metric_Pad1.33x1.80mm_HandSolder, F.Cu at (206.0, 138.3)
- added C57: 100nF, Capacitor_SMD:C_1206_3216Metric_Pad1.33x1.80mm_HandSolder, F.Cu at (249.1, 67.3)
- added C58: 100nF, Capacitor_SMD:C_1206_3216Metric_Pad1.33x1.80mm_HandSolder, F.Cu at (249.1, 70.7)
- added C59: 220nF, Capacitor_SMD:C_1206_3216Metric_Pad1.33x1.80mm_HandSolder, F.Cu at (249.1, 74.0)
- added C60: 220nF, Capacitor_SMD:C_1206_3216Metric_Pad1.33x1.80mm_HandSolder, F.Cu at (249.1, 77.3)
- added C61: 4.7μF, Capacitor_SMD:C_1206_3216Metric_Pad1.33x1.80mm_HandSolder, F.Cu at (249.1, 80.7)
- added C62: 100nF, Capacitor_SMD:C_1206_3216Metric_Pad1.33x1.80mm_HandSolder, F.Cu at (249.1, 84.0)
- added C63: 100nF, Capacitor_SMD:C_1206_3216Metric_Pad1.33x1.80mm_HandSolder, F.Cu at (249.1, 87.4)
- added C64: 100nF, Capacitor_SMD:C_1206_3216Metric_Pad1.33x1.80mm_HandSolder, F.Cu at (249.1, 92.8)
- added C65: 100nF, Capacitor_SMD:C_1206_3216Metric_Pad1.33x1.80mm_HandSolder, F.Cu at (249.1, 96.1)
- added C66: 220nF, Capacitor_SMD:C_1206_3216Metric_Pad1.33x1.80mm_HandSolder, F.Cu at (249.1, 99.5)
- added C67: 220nF, Capacitor_SMD:C_1206_3216Metric_Pad1.33x1.80mm_HandSolder, F.Cu at (249.1, 102.8)
- added C68: 4.7μF, Capacitor_SMD:C_1206_3216Metric_Pad1.33x1.80mm_HandSolder, F.Cu at (249.1, 106.2)
- added C69: 100nF, Capacitor_SMD:C_1206_3216Metric_Pad1.33x1.80mm_HandSolder, F.Cu at (249.1, 109.5)
- added C70: 100nF, Capacitor_SMD:C_1206_3216Metric_Pad1.33x1.80mm_HandSolder, F.Cu at (249.1, 112.8)
- added C71: 100nF, Capacitor_SMD:C_1206_3216Metric_Pad1.33x1.80mm_HandSolder, F.Cu at (227.6, 67.3)
- added C72: 100nF, Capacitor_SMD:C_1206_3216Metric_Pad1.33x1.80mm_HandSolder, F.Cu at (227.6, 70.7)
- added C73: 220nF, Capacitor_SMD:C_1206_3216Metric_Pad1.33x1.80mm_HandSolder, F.Cu at (227.6, 74.0)
- added C74: 220nF, Capacitor_SMD:C_1206_3216Metric_Pad1.33x1.80mm_HandSolder, F.Cu at (227.6, 77.3)
- added C75: 4.7μF, Capacitor_SMD:C_1206_3216Metric_Pad1.33x1.80mm_HandSolder, F.Cu at (227.6, 80.7)
- added C76: 100nF, Capacitor_SMD:C_1206_3216Metric_Pad1.33x1.80mm_HandSolder, F.Cu at (227.6, 84.0)
- added C77: 100nF, Capacitor_SMD:C_1206_3216Metric_Pad1.33x1.80mm_HandSolder, F.Cu at (227.6, 87.4)
- added M1: Stepper_Motor_unipolar_6pin, Connector_JST:JST_PH_B6B-PH-K_1x06_P2.00mm_Vertical, F.Cu at (131.0, 133.0)
- added M2: Stepper_Motor_unipolar_6pin, Connector_JST:JST_PH_B6B-PH-K_1x06_P2.00mm_Vertical, F.Cu at (188.0, 74.9)
- added M3: Stepper_Motor_unipolar_6pin, Connector_JST:JST_PH_B6B-PH-K_1x06_P2.00mm_Vertical, F.Cu at (188.0, 81.5)
- added M4: Stepper_Motor_unipolar_6pin, Connector_JST:JST_PH_B6B-PH-K_1x06_P2.00mm_Vertical, F.Cu at (188.0, 88.0)
- added M5: Stepper_Motor_unipolar_6pin, Connector_JST:JST_PH_B6B-PH-K_1x06_P2.00mm_Vertical, F.Cu at (188.0, 94.5)
- added M6: Stepper_Motor_unipolar_6pin, Connector_JST:JST_PH_B6B-PH-K_1x06_P2.00mm_Vertical, F.Cu at (188.0, 101.1)
- added M7: Stepper_Motor_unipolar_6pin, Connector_JST:JST_PH_B6B-PH-K_1x06_P2.00mm_Vertical, F.Cu at (188.0, 107.7)
- added M8: Stepper_Motor_unipolar_6pin, Connector_JST:JST_PH_B6B-PH-K_1x06_P2.00mm_Vertical, F.Cu at (188.0, 114.2)
- added R11: 50mΩ, Resistor_SMD:R_1206_3216Metric_Pad1.30x1.75mm_HandSolder, F.Cu at (127.0, 132.5)
- added R12: 50mΩ, Resistor_SMD:R_1206_3216Metric_Pad1.30x1.75mm_HandSolder, F.Cu at (127.0, 123.5)
- added R13: 10kΩ, Resistor_SMD:R_1206_3216Metric_Pad1.30x1.75mm_HandSolder, F.Cu at (110.8, 139.8)
- added R14: 10kΩ, Resistor_SMD:R_1206_3216Metric_Pad1.30x1.75mm_HandSolder, F.Cu at (110.8, 143.1)
- added R15: 50kΩ, Resistor_SMD:R_1206_3216Metric_Pad1.30x1.75mm_HandSolder, F.Cu at (110.8, 146.4)
- added R16: 50mΩ, Resistor_SMD:R_1206_3216Metric_Pad1.30x1.75mm_HandSolder, F.Cu at (209.4, 33.0)
- added R17: 50mΩ, Resistor_SMD:R_1206_3216Metric_Pad1.30x1.75mm_HandSolder, F.Cu at (209.4, 36.3)
- added R18: 10kΩ, Resistor_SMD:R_1206_3216Metric_Pad1.30x1.75mm_HandSolder, F.Cu at (209.4, 39.6)
- added R19: 10kΩ, Resistor_SMD:R_1206_3216Metric_Pad1.30x1.75mm_HandSolder, F.Cu at (209.4, 43.0)
- added R20: 50kΩ, Resistor_SMD:R_1206_3216Metric_Pad1.30x1.75mm_HandSolder, F.Cu at (209.4, 46.3)
- added R21: 50mΩ, Resistor_SMD:R_1206_3216Metric_Pad1.30x1.75mm_HandSolder, F.Cu at (233.5, 118.2)
- added R22: 50mΩ, Resistor_SMD:R_1206_3216Metric_Pad1.30x1.75mm_HandSolder, F.Cu at (233.5, 121.5)
- added R23: 10kΩ, Resistor_SMD:R_1206_3216Metric_Pad1.30x1.75mm_HandSolder, F.Cu at (233.5, 124.8)
- added R24: 10kΩ, Resistor_SMD:R_1206_3216Metric_Pad1.30x1.75mm_HandSolder, F.Cu at (233.5, 128.1)
- added R25: 50kΩ, Resistor_SMD:R_1206_3216Metric_Pad1.30x1.75mm_HandSolder, F.Cu at (233.5, 131.4)
- added R26: 50mΩ, Resistor_SMD:R_1206_3216Metric_Pad1.30x1.75mm_HandSolder, F.Cu at (212.0, 92.7)
- added R27: 50mΩ, Resistor_SMD:R_1206_3216Metric_Pad1.30x1.75mm_HandSolder, F.Cu at (212.0, 96.0)
- added R28: 10kΩ, Resistor_SMD:R_1206_3216Metric_Pad1.30x1.75mm_HandSolder, F.Cu at (212.0, 99.3)
- added R29: 10kΩ, Resistor_SMD:R_1206_3216Metric_Pad1.30x1.75mm_HandSolder, F.Cu at (212.0, 102.7)
- added R30: 50kΩ, Resistor_SMD:R_1206_3216Metric_Pad1.30x1.75mm_HandSolder, F.Cu at (212.0, 106.0)
- added R31: 50mΩ, Resistor_SMD:R_1206_3216Metric_Pad1.30x1.75mm_HandSolder, F.Cu at (212.0, 118.2)
- added R32: 50mΩ, Resistor_SMD:R_1206_3216Metric_Pad1.30x1.75mm_HandSolder, F.Cu at (212.0, 121.5)
- added R33: 10kΩ, Resistor_SMD:R_1206_3216Metric_Pad1.30x1.75mm_HandSolder, F.Cu at (212.0, 124.8)
- added R34: 10kΩ, Resistor_SMD:R_1206_3216Metric_Pad1.30x1.75mm_HandSolder, F.Cu at (212.0, 128.1)
- added R35: 50kΩ, Resistor_SMD:R_1206_3216Metric_Pad1.30x1.75mm_HandSolder, F.Cu at (212.0, 131.4)
- added R36: 50mΩ, Resistor_SMD:R_1206_3216Metric_Pad1.30x1.75mm_HandSolder, F.Cu at (255.1, 67.3)
- added R37: 50mΩ, Resistor_SMD:R_1206_3216Metric_Pad1.30x1.75mm_HandSolder, F.Cu at (255.1, 70.6)
- added R38: 10kΩ, Resistor_SMD:R_1206_3216Metric_Pad1.30x1.75mm_HandSolder, F.Cu at (255.1, 73.9)
- added R39: 10kΩ, Resistor_SMD:R_1206_3216Metric_Pad1.30x1.75mm_HandSolder, F.Cu at (255.1, 77.2)
- added R40: 50kΩ, Resistor_SMD:R_1206_3216Metric_Pad1.30x1.75mm_HandSolder, F.Cu at (255.1, 80.5)
- added R41: 50mΩ, Resistor_SMD:R_1206_3216Metric_Pad1.30x1.75mm_HandSolder, F.Cu at (255.1, 92.7)
- added R42: 50mΩ, Resistor_SMD:R_1206_3216Metric_Pad1.30x1.75mm_HandSolder, F.Cu at (255.1, 96.0)
- added R43: 10kΩ, Resistor_SMD:R_1206_3216Metric_Pad1.30x1.75mm_HandSolder, F.Cu at (255.1, 99.3)
- added R44: 10kΩ, Resistor_SMD:R_1206_3216Metric_Pad1.30x1.75mm_HandSolder, F.Cu at (255.1, 102.7)
- added R45: 50kΩ, Resistor_SMD:R_1206_3216Metric_Pad1.30x1.75mm_HandSolder, F.Cu at (255.1, 106.0)
- added R46: 50mΩ, Resistor_SMD:R_1206_3216Metric_Pad1.30x1.75mm_HandSolder, F.Cu at (233.5, 67.3)
- added R47: 50mΩ, Resistor_SMD:R_1206_3216Metric_Pad1.30x1.75mm_HandSolder, F.Cu at (233.5, 70.6)
- added R48: 10kΩ, Resistor_SMD:R_1206_3216Metric_Pad1.30x1.75mm_HandSolder, F.Cu at (233.5, 73.9)
- added R49: 10kΩ, Resistor_SMD:R_1206_3216Metric_Pad1.30x1.75mm_HandSolder, F.Cu at (233.5, 77.2)
- added R50: 50kΩ, Resistor_SMD:R_1206_3216Metric_Pad1.30x1.75mm_HandSolder, F.Cu at (233.5, 80.5)
- added U10: A4988SETTR-T, Package_DFN_QFN:VQFN-28-1EP_5x5mm_P0.5mm_EP3.25x3.25mm_ThermalVias, F.Cu at (240.5, 120.2)
- added U11: A4988SETTR-T, Package_DFN_QFN:VQFN-28-1EP_5x5mm_P0.5mm_EP3.25x3.25mm_ThermalVias, F.Cu at (218.9, 94.7)
- added U12: A4988SETTR-T, Package_DFN_QFN:VQFN-28-1EP_5x5mm_P0.5mm_EP3.25x3.25mm_ThermalVias, F.Cu at (218.9, 120.2)
- added U13: A4988SETTR-T, Package_DFN_QFN:VQFN-28-1EP_5x5mm_P0.5mm_EP3.25x3.25mm_ThermalVias, F.Cu at (262.1, 69.2)
- added U14: A4988SETTR-T, Package_DFN_QFN:VQFN-28-1EP_5x5mm_P0.5mm_EP3.25x3.25mm_ThermalVias, F.Cu at (262.1, 94.7)
- added U15: A4988SETTR-T, Package_DFN_QFN:VQFN-28-1EP_5x5mm_P0.5mm_EP3.25x3.25mm_ThermalVias, F.Cu at (240.5, 69.2)
- added U8: A4988SETTR-T, Package_DFN_QFN:VQFN-28-1EP_5x5mm_P0.5mm_EP3.25x3.25mm_ThermalVias, F.Cu at (120.2, 128.0)
- added U9: A4988SETTR-T, Package_DFN_QFN:VQFN-28-1EP_5x5mm_P0.5mm_EP3.25x3.25mm_ThermalVias, F.Cu at (216.4, 35.0)
Routing:
- net /Motors & Drivers/Driver 1/1B: track 0.00 -> 11.1 mm, vias 0 -> 1
- net /Motors & Drivers/Driver 1/2B: track 0.00 -> 10.4 mm
- net /Motors & Drivers/Driver 1/1A: track 0.00 -> 10.2 mm
- net /Motors & Drivers/Driver 1/2A: track 0.00 -> 8.57 mm
- net Net-(U8-CP2): track 0.00 -> 5.44 mm
- net Net-(U8-SENSE2): track 0.00 -> 5.17 mm
- net Net-(U8-SENSE1): track 0.00 -> 5.17 mm
- net GND: track 40.8 -> 44.6 mm, vias 48 -> 54
- net Net-(U8-CP1): track 0.00 -> 2.11 mm
- net Net-(U8-VCP): track 0.00 -> 1.97 mm
Other:
- board size 70 x 100 mm -> 75 x 105 mm

Commit message: Update stepper_music.kicad_pcb
Parts:
- moved M2 65.9 mm to (131.0, 108.0), turned to 90 degrees
- moved M4 64.4 mm to (131.0, 58.0), turned to 90 degrees
- moved M3 57.0 mm to (131.0, 83.0), turned to 90 degrees
- moved R15 18.6 mm to (127.8, 138.9)
- moved R14 17.1 mm to (127.8, 141.3)
- moved R13 7.38 mm to (114.5, 133.4), turned to 90 degrees
- moved C26 5.71 mm to (122.0, 134.4), turned to -90 degrees
- moved TP2 3.43 mm to (89.8, 140.4)
Routing:
- net /~{SLEEP}: track 0.00 -> 69.8 mm, vias 0 -> 2
- net /~{RESET}: track 0.00 -> 68.8 mm, vias 0 -> 2
- net /MS3: track 3.43 -> 64.8 mm, vias 0 -> 2
- net /MS2: track 3.36 -> 63.3 mm, vias 0 -> 2
- net /MS1: track 3.32 -> 61.9 mm, vias 0 -> 2
- net /STEP_1: track 0.00 -> 53.7 mm
- net /DIR_1: track 0.00 -> 48.8 mm
- net /~{ENABLE_3}: track 0.00 -> 22.2 mm
- net /~{ENABLE_4}: track 0.00 -> 21.5 mm
- net /DIR_8: track 0.00 -> 21.3 mm
- net /DIR_7: track 0.00 -> 21.2 mm
- net /~{ENABLE_5}: track 0.00 -> 20.8 mm
- net /STEP_4: track 0.00 -> 18.2 mm
- net Net-(U8-REF): track 0.00 -> 16.2 mm, vias 0 -> 2
- net /DIR_6: track 3.28 -> 18.8 mm
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- added copper zone on F.Cu, net Net-(U8-VREG)

Commit message: !!!!!
Parts:
- moved R42 190.4 mm to (75.5, 33.0), turned to 180 degrees
- moved U14 190.2 mm to (80.0, 39.8)
- moved C70 190.1 mm to (75.5, 35.5), turned to 180 degrees
- moved C64 183.3 mm to (74.0, 38.8), turned to 180 degrees
- moved C65 183.2 mm to (74.3, 41.4)
- moved R41 180.8 mm to (84.5, 33.0)
- moved C66 180.7 mm to (76.8, 45.2), turned to -90 degrees
- moved C69 180.5 mm to (84.5, 35.5)
- moved R45 179.6 mm to (90.8, 33.5), turned to 90 degrees
- moved R44 179.1 mm to (85.4, 45.5), turned to 180 degrees
- moved C68 176.4 mm to (86.4, 38.0)
- moved C67 174.3 mm to (85.4, 43.0)
- moved R43 174.0 mm to (90.8, 42.2), turned to 90 degrees
- moved R50 172.4 mm to (63.5, 52.2), turned to 180 degrees
- moved U15 170.8 mm to (69.8, 63.0), turned to 90 degrees
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Connections:
- U1 pad 2: /~{ENABLE_6} -> /ENABLE_6
- U1 pad 3: /~{ENABLE_7} -> /ENABLE_7
- U1 pad 39: /~{ENABLE_1} -> /ENABLE_1
- U1 pad 4: /~{ENABLE_8} -> /ENABLE_8
- U1 pad 40: /~{ENABLE_2} -> /ENABLE_2
- U1 pad 51: /~{ENABLE_3} -> /ENABLE_3
- U1 pad 52: /~{ENABLE_4} -> /ENABLE_4
- U1 pad 53: /~{ENABLE_5} -> /ENABLE_5
- U10 pad 2: /Motors & Drivers/~{ENABLE_3} -> /ENABLE_3
- U11 pad 2: /Motors & Drivers/~{ENABLE_4} -> /ENABLE_4
- U12 pad 2: /Motors & Drivers/~{ENABLE_5} -> /ENABLE_5
- U13 pad 2: /Motors & Drivers/~{ENABLE_6} -> /ENABLE_6
- U14 pad 2: /Motors & Drivers/~{ENABLE_7} -> /ENABLE_7
- U15 pad 2: /Motors & Drivers/~{ENABLE_8} -> /ENABLE_8
- U8 pad 2: /Motors & Drivers/~{ENABLE_1} -> /ENABLE_1
- U9 pad 2: /Motors & Drivers/~{ENABLE_2} -> /ENABLE_2
Routing:
- net /MS1: track 61.9 -> 266.6 mm, vias 2 -> 9
- net /~{SLEEP}: track 69.8 -> 272.5 mm, vias 2 -> 9
- net /MS2: track 63.3 -> 262.3 mm, vias 2 -> 9
- net /MS3: track 64.8 -> 257.8 mm, vias 2 -> 9
- net /~{RESET}: track 68.8 -> 260.2 mm, vias 2 -> 9
- net /ENABLE_5: track 0.00 -> 169.8 mm, vias 0 -> 2
- net /ENABLE_7: track 0.00 -> 168.5 mm, vias 0 -> 2
- net /ENABLE_6: track 0.00 -> 163.2 mm, vias 0 -> 2
- net /STEP_7: track 0.00 -> 151.2 mm, vias 0 -> 2
- net /ENABLE_4: track 0.00 -> 148.2 mm, vias 0 -> 2
- net /STEP_8: track 0.00 -> 143.5 mm, vias 0 -> 2
- net /DIR_6: track 18.8 -> 153.7 mm
- net /ENABLE_8: track 0.00 -> 133.4 mm, vias 0 -> 2
- net /DIR_7: track 21.2 -> 146.3 mm, vias 0 -> 2
- net /ENABLE_3: track 0.00 -> 125.0 mm, vias 0 -> 2
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- added copper zone on F.Cu, net Net-(U10-VREG)
- added copper zone on F.Cu, net Net-(U11-VREG)
- added copper zone on F.Cu, net Net-(U12-VREG)
- added copper zone on F.Cu, net Net-(U13-VREG)
- added copper zone on F.Cu, net Net-(U14-VREG)
- added copper zone on F.Cu, net Net-(U15-VREG)
- added copper zone on F.Cu, net Net-(U9-VREG)
Other:
- board size 75 x 105 mm -> 75 x 155 mm
