File: pcb/stepper_music.kicad_pcb (KiCad board)
At the start: 4 copper layers, 75 x 155 mm, 162 parts, among them J1 USB_C_Receptacle, J2 Conn_ST_STDC14, J3 MIDI IN, J4 MIDI THRU, J5 Conn_01x02, M1 Stepper_Motor_unipolar_6pin, M2 Stepper_Motor_unipolar_6pin, M3 Stepper_Motor_unipolar_6pin, M4 Stepper_Motor_unipolar_6pin, M5 Stepper_Motor_unipolar_6pin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

Commit message: w
Parts:
- moved TP1 59.9 mm to (89.0, 176.0)
- moved TP2 0.60 mm to (85.0, 176.0)
Routing:
- net +3.3V: track 6.87 -> 14.9 mm, vias 18 -> 44
- net GND: track 94.0 -> 96.0 mm, vias 160 -> 164
- net /STEP_5: track 127.1 -> 126.5 mm
- net +12V: vias 51 -> 83
- added copper zone on In2.Cu, net +12V
- added copper zone on In2.Cu, net +3.3V

Commit message: w
Parts:
- added LG1: UCSB_IEEE, footprints:UCSB_IEEE_Logo, F.Cu at (92.6, 64.5)
- added LG2: UCSB, footprints:UCSB_Medium, F.Cu at (92.8, 78.5)
Routing:
- net GND: track 96.0 -> 97.3 mm
- net +12V: vias 83 -> 110
Other:
- board text added: "8x Stepper Motor Music Controller Revision 1.0 Designed By: Kyle Schmerge"
