File: pcb/stepper_music.kicad_pcb (KiCad board)
At the start: 4 copper layers, 75 x 155 mm, 164 parts, among them J1 USB_C_Receptacle, J2 Conn_ST_STDC14, J3 MIDI IN, J4 MIDI THRU, J5 Conn_01x02, M1 Stepper_Motor_unipolar_6pin, M2 Stepper_Motor_unipolar_6pin, M3 Stepper_Motor_unipolar_6pin, M4 Stepper_Motor_unipolar_6pin, M5 Stepper_Motor_unipolar_6pin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

Commit message: name
Other:
- board text added: "+12V"
- board text added: "+3.3V"
- board text added: "+5V"
- board text added: "GND"
Changed lines of the file:
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@@
 		(property "Reference" "TP4"
 			(at 0 -1.648 0)
-			(layer "F.SilkS")
+			(layer "User.1")
 			(effects
 				(font
@@
 		(property "Reference" "TP2"
 			(at 0 -1.648 0)
-			(layer "F.SilkS")
+			(layer "User.1")
 			(effects
 				(font
@@
 		(property "Reference" "TP1"
 			(at 0 -1.648 0)
-			(layer "F.SilkS")
+			(layer "User.1")
 			(effects
 				(font
@@
 		(property "Reference" "TP3"
 			(at 0 -1.648 0)
-			(layer "F.SilkS")
+			(layer "User.1")
 			(effects
 				(font
@@
 		(layer "Edge.Cuts")
 	)
+	(gr_text "+12V"
+		(at 76.5 100.5 0)
+		(layer "F.SilkS")
+		(effects
+			(font
+				(size 1 1)
+				(thickness 0.1)
+			)
+		)
+	)
+	(gr_text "+3.3V"
+		(at 85 174 0)
+		(layer "F.SilkS")
+		(effects
+			(font
+				(size 1 1)
+				(thickness 0.1)
+			)
+		)
+	)
+	(gr_text "GND"
+		(at 89 174 0)
+		(layer "F.SilkS")
+		(effects
+			(font
+				(size 1 1)
+				(thickness 0.1)
+			)
+		)
+	)
+	(gr_text "+5V"
+		(at 101.5 132 0)
+		(layer "F.SilkS")
+		(effects
+			(font
+				(size 1 1)
+				(thickness 0.1)
+			)
+		)
+	)
 	(gr_text "8x Stepper Motor Music Controller\nRevision 1.0\nDesigned By:\nKyle Schmerge"
 		(at 92.375 107.25 90)
@@
 		(hatch edge 0.5)
 		(priority 1)
-		(connect_pads yes
+		(connect_pads
 			(clearance 0.1)
 		)
 		(min_thickness 0.25)
 		(fill yes
-			(thermal_gap 0.5)
+			(thermal_gap 0.1)
 			(thermal_bridge_width 0.5)
 			(island_removal_mode 0)

Commit message: holes
Parts:
- added H1: Hole, MountingHole:MountingHole_3.2mm_M3_DIN965, F.Cu at (60.0, 30.0)
- added H2: Hole, MountingHole:MountingHole_3.2mm_M3_DIN965, F.Cu at (125.0, 30.0)
- added H3: Hole, MountingHole:MountingHole_3.2mm_M3_DIN965, F.Cu at (60.0, 175.0)
- added H4: Hole, MountingHole:MountingHole_3.2mm_M3_DIN965, F.Cu at (125.0, 175.0)
- moved R15 9.52 mm to (112.8, 177.5)
Routing:
- net Net-(U8-REF): track 14.9 -> 17.0 mm
