File: pcb/driver.kicad_sch (KiCad schematic)
At the start: 13 parts, among them U8 A4988SETTR-T

Commit message: w
Parts:
- C22, C25: Manufacturer Part Number (none) -> C1206C224K5RACTU; Vendor Part Number (none) -> 399-C1206C224K5RACTUCT-ND
- C26: Manufacturer Part Number (none) -> CL31B475KAHNNNE; Vendor Part Number (none) -> 1276-1055-1-ND
- R11, R12: Manufacturer Part Number (none) -> CSR1206FT50L0; Vendor Part Number (none) -> CSR1206FT50L0CT-ND
- R15: Manufacturer Part Number (none) -> RT1206BRD0750KL; Vendor Part Number (none) -> 13-RT1206BRD0750KLCT-ND
- U8: Manufacturer Part Number (none) -> A4988SETTR-T; Vendor (none) -> Digi-Key; Vendor Part Number (none) -> 620-1343-1-ND
Changed lines of the file:
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@@
 			)
 		)
-		(property "Manufacturer Part Number" ""
+		(property "Manufacturer Part Number" "C1206C224K5RACTU"
 			(at 179.07 82.55 0)
 			(hide yes)
@@
 			)
 		)
-		(property "Vendor Part Number" ""
+		(property "Vendor Part Number" "399-C1206C224K5RACTUCT-ND"
 			(at 179.07 82.55 0)
 			(hide yes)
@@
 			)
 		)
-		(property "Manufacturer Part Number" ""
+		(property "Manufacturer Part Number" "CSR1206FT50L0"
 			(at 91.44 118.11 0)
 			(hide yes)
@@
 			)
 		)
-		(property "Vendor Part Number" ""
+		(property "Vendor Part Number" "CSR1206FT50L0CT-ND"
 			(at 91.44 118.11 0)
 			(hide yes)
@@
 			)
 		)
-		(property "Manufacturer Part Number" ""
+		(property "Manufacturer Part Number" "CSR1206FT50L0"
 			(at 80.01 118.11 0)
 			(hide yes)
@@
 			)
 		)
-		(property "Vendor Part Number" ""
+		(property "Vendor Part Number" "CSR1206FT50L0CT-ND"
 			(at 80.01 118.11 0)
 			(hide yes)
@@
 			)
 		)
+		(property "Manufacturer Part Number" "A4988SETTR-T"
+			(at 127 102.87 0)
+			(hide yes)
+			(show_name no)
+			(do_not_autoplace no)
+			(effects
+				(font
+					(size 1.27 1.27)
+				)
+			)
+		)
+		(property "Vendor" "Digi-Key"
+			(at 127 102.87 0)
+			(hide yes)
+			(show_name no)
+			(do_not_autoplace no)
+			(effects
+				(font
+					(size 1.27 1.27)
+				)
+			)
+		)
+		(property "Vendor Part Number" "620-1343-1-ND"
+			(at 127 102.87 0)
+			(hide yes)
+			(show_name no)
+			(do_not_autoplace no)
+			(effects
+				(font
+					(size 1.27 1.27)
+				)
+			)
+		)
 		(pin "19"
 		)
@@
 			)
 		)
-		(property "Manufacturer Part Number" ""
+		(property "Manufacturer Part Number" "CL31B475KAHNNNE"
 			(at 193.04 82.55 0)
 			(hide yes)
@@
 			)
 		)
-		(property "Vendor Part Number" ""
+		(property "Vendor Part Number" "1276-1055-1-ND"
 			(at 193.04 82.55 0)
 			(hide yes)
@@
 			)
 		)
-		(property "Manufacturer Part Number" ""
+		(property "Manufacturer Part Number" "C1206C224K5RACTU"
 			(at 165.1 124.46 0)
 			(hide yes)
@@
 			)
 		)
-		(property "Vendor Part Number" ""
+		(property "Vendor Part Number" "399-C1206C224K5RACTUCT-ND"
 			(at 165.1 124.46 0)
 			(hide yes)
@@
 			)
 		)
-		(property "Manufacturer Part Number" ""
+		(property "Manufacturer Part Number" "RT1206BRD0750KL"
 			(at 106.68 76.2 0)
 			(hide yes)
@@
 			)
 		)
-		(property "Vendor Part Number" ""
+		(property "Vendor Part Number" "13-RT1206BRD0750KLCT-ND"
 			(at 106.68 76.2 0)
 			(hide yes)
