File: pcb/stepper_music.kicad_sch (KiCad schematic)
At the start: 17 parts, among them J1 USB_C_Receptacle, J2 Conn_ST_STDC14, U1 STM32F401RCTx, Y1 Crystal

Commit message: work
Parts:
- added C11, C12, C14, C17, C18: 100nF, Capacitor_SMD:C_1206_3216Metric_Pad1.33x1.80mm_HandSolder, symbol Device:C
- added C13, C16, C19, C21: 10μF, Capacitor_SMD:C_1206_3216Metric_Pad1.33x1.80mm_HandSolder, symbol Device:C
- added C15: 2.2μF, Capacitor_SMD:C_1206_3216Metric_Pad1.33x1.80mm_HandSolder, symbol Device:C
- added C20: 1μF, Capacitor_SMD:C_1206_3216Metric_Pad1.33x1.80mm_HandSolder, symbol Device:C
- added D1: 1N914, Diode_SMD:D_SOD-523, symbol Diode:1N914
- added J3: MIDI IN, footprints:KYCON_KCDX-5S-N, symbol Connector:DIN-5_180degree
- added J4: MIDI THRU, footprints:KYCON_KCDX-5S-N, symbol Connector:DIN-5_180degree
- added J5: Conn_01x02, Connector_AMASS:AMASS_XT30PW-M_1x02_P2.50mm_Horizontal, symbol Connector_Generic:Conn_01x02
- added L1: 4.7μH, Inductor_SMD:L_1008_2520Metric_Pad1.43x2.20mm_HandSolder, symbol Device:L
- added R10, R4, R9: 220Ω, Resistor_SMD:R_1206_3216Metric_Pad1.30x1.75mm_HandSolder, symbol Device:R_US
- added R5: 10kΩ, Resistor_SMD:R_1206_3216Metric_Pad1.30x1.75mm_HandSolder, symbol Device:R_US
- added R6: 1kΩ, Resistor_SMD:R_1206_3216Metric_Pad1.30x1.75mm_HandSolder, symbol Device:R_US
- added R7: 88.7kΩ, Resistor_SMD:R_1206_3216Metric_Pad1.30x1.75mm_HandSolder, symbol Device:R_US
- added R8: 22.1kΩ, Resistor_SMD:R_1206_3216Metric_Pad1.30x1.75mm_HandSolder, symbol Device:R_US
- added TP1: GND, TestPoint:TestPoint_Pad_D1.5mm, symbol Connector:TestPoint
- added TP2: +3.3V, TestPoint:TestPoint_Pad_D1.5mm, symbol Connector:TestPoint
- added TP3: +5V, TestPoint:TestPoint_Pad_D1.5mm, symbol Connector:TestPoint
- added TP4: +12V, TestPoint:TestPoint_Pad_D1.5mm, symbol Connector:TestPoint
- added U2: 6N138, Package_SO:SOIC-8_3.9x4.9mm_P1.27mm, symbol Isolator:6N138
- added U3: LD1117S33TR_SOT223, Package_TO_SOT_SMD:SOT-223-3_TabPin2, symbol Regulator_Linear:LD1117S33TR_SOT223
- added U4: LMR50410, Package_TO_SOT_SMD:SOT-23-6, symbol Regulator_Switching:LMR50410
- added U5: SN74LV1T34DBV, Package_TO_SOT_SMD:SOT-23-5, symbol Logic_LevelTranslator:SN74LV1T34DBV
- added U6, U7: LM66100DCK, Package_TO_SOT_SMD:SOT-363_SC-70-6, symbol Power_Management:LM66100DCK
- C1, C2: value ?pF -> 18pF; footprint (none) -> Capacitor_SMD:C_0402_1005Metric; Manufacturer Part Number (none) -> GJM1555C1H180GB01D; Vendor (none) -> Digi-Key; Vendor Part Number (none) -> 490-8082-1-ND
- C10, C3, C5, C6, C7, C8: footprint (none) -> Capacitor_SMD:C_1206_3216Metric_Pad1.33x1.80mm_HandSolder; Manufacturer Part Number (none) -> 1206B104K500CT; Vendor (none) -> Digi-Key; Vendor Part Number (none) -> 1292-1605-1-ND
- C4: footprint (none) -> Capacitor_SMD:C_1206_3216Metric_Pad1.33x1.80mm_HandSolder; Manufacturer Part Number (none) -> CL31B105KAHNNNE; Vendor (none) -> Digi-Key; Vendor Part Number (none) -> 1276-1097-1-ND
- C9: footprint (none) -> Capacitor_SMD:C_1206_3216Metric_Pad1.33x1.80mm_HandSolder; Manufacturer Part Number (none) -> UMK316BJ225KD-T; Vendor (none) -> Digi-Key; Vendor Part Number (none) -> 587-2402-1-ND
- J1: footprint (none) -> footprints:USB_C_Receptacle_short; Manufacturer Part Number (none) -> USB4056-03-A; Vendor (none) -> Digi-Key; Vendor Part Number (none) -> 2073-USB4056-03-ACT-ND
- J2: footprint (none) -> Connector_PinHeader_1.27mm:PinHeader_2x07_P1.27mm_Vertical_SMD; Manufacturer Part Number (none) -> FTSH-107-01-L-DV-K; Vendor (none) -> Digi-Key; Vendor Part Number (none) -> SAM9449-ND
- R1, R2, R3: footprint (none) -> Resistor_SMD:R_1206_3216Metric_Pad1.30x1.75mm_HandSolder; Vendor (none) -> Digi-Key
- U1: Manufacturer Part Number (none) -> STM32F401RCT6; Vendor (none) -> Digi-Key; Vendor Part Number (none) -> 497-14047-ND
- Y1: value Crystal -> 25MHz; footprint (none) -> Crystal:Crystal_SMD_HC49-SD; Manufacturer Part Number (none) -> ECS-250-18-5PX-F-TR; Vendor (none) -> Digi-Key; Vendor Part Number (none) -> XC1305CT-ND
Connections:
- net +3.3V: now also C13.1, R6.1, TP2.1, U3.2 (VO)
- net +5V: now also C12.1, C17.1, C18.1, C19.1, R9.2, TP3.1, U2.8 (VCC), U3.3 (VI), U5.5 (VCC), U6.6 (VOUT), U7.6 (VOUT); no longer J1.A4 (VBUS), J1.A9 (VBUS), J1.B4 (VBUS), J1.B9 (VBUS)
- net GND: now also C11.2, C12.2, C13.2, C15.2, C16.2, C17.2, C18.2, C19.2, C20.2, C21.2, J4.2, J5.1 (Pin_1), R5.2, R8.2, TP1.1, U2.5 (GND), U3.1 (GND), U4.2 (GND), U5.3 (GND), U6.2 (GND), U7.2 (GND)
- net MS1: now also U1.26 (PB0)
- net MS2: now also U1.27 (PB1)
- net MS3: now also U1.28 (PB2)
- net ~{RESET}: now also U1.56 (PB4)
- net ~{SLEEP}: now also U1.57 (PB5)
- net ~{RST}: now reaches C10.1, R3.2, U1.7 (NRST)
- net ~{RST}: now also J2.12 (~{RST})
- net ~{ENABLE_6}: now reaches U1.2 (PC13)
- net ~{ENABLE_7}: now reaches U1.3 (PC14)
- net ~{ENABLE_1}: now reaches U1.39 (PC8)
- net ~{ENABLE_8}: now reaches U1.4 (PC15)
- net ~{ENABLE_2}: now reaches U1.40 (PC9)
- net MIDI_RX: now reaches U1.43 (PA10)
- net MIDI_RX: now also R6.2, U2.6 (VO2), U5.2 (A)
- net SWDIO: now reaches U1.46 (PA13)
- net SWDIO: now also J2.4 (JTMS/SWDIO)
- net SWCLK: now reaches U1.49 (PA14)
- net SWCLK: now also J2.6 (JCLK/SWCLK)
- net ~{ENABLE_3}: now reaches U1.51 (PC10)
- net ~{ENABLE_4}: now reaches U1.52 (PC11)
- net ~{ENABLE_5}: now reaches U1.53 (PC12)
- net SWO: now reaches U1.55 (PB3)
- net SWO: now also J2.8 (JTDO/SWO)
- new net: R10.2, U5.4 (Y)
- new net: C11.1, J3.2
- new net: C16.1, L1.2, R7.2, U6.1 (VIN), U7.3 (~{CE})
- new net: R7.1, R8.1, U4.3 (FB)
- new net: J3.4, R4.1
- new net: D1.1 (K), R4.2, U2.2 (C1)
- new net: D1.2 (A), J3.5, U2.3 (C2)
- new net: C14.1, U4.1 (CB)
- new net: C14.2, L1.1, U4.6 (SW)
- new net: R5.1, U2.7 (VO1)
- new net: J4.4, R9.1
- new net: J4.5, R10.1
- new net +12V: C15.1, C21.1, J5.2 (Pin_2), TP4.1, U4.4 (EN), U4.5 (VIN)
- new net VBUS: C20.1, J1.A4 (VBUS), J1.A9 (VBUS), J1.B4 (VBUS), J1.B9 (VBUS), U6.3 (~{CE}), U7.1 (VIN)
- no-connect marks 10 -> 33
Other:
- moved on the sheet: C1, C10, C2, C3, C4, C5, C6, C7, C8, C9, J1, J2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

Commit message: w
Parts:
- R1, R2: Manufacturer Part Number (none) -> RC1206FR-075K1L; Vendor Part Number (none) -> 311-5.10KFRCT-ND
- R10, R4, R9: Manufacturer Part Number (none) -> RMCF1206FT220R; Vendor Part Number (none) -> RMCF1206FT220RCT-ND
- R3, R5: Manufacturer Part Number (none) -> RMCF1206FT10K0; Vendor Part Number (none) -> RMCF1206FT10K0CT-ND
- R6: Manufacturer Part Number (none) -> RC1206FR-071KL; Vendor Part Number (none) -> 311-1.00KFRCT-ND
- R7: Manufacturer Part Number (none) -> RC1206FR-0788K7L; Vendor Part Number (none) -> 311-88.7KFRCT-ND
- R8: Manufacturer Part Number (none) -> CRCW120622K1FKEAC; Vendor Part Number (none) -> 541-CRCW120622K1FKEACCT-ND
Changed lines of the file:
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@@
 			)
 		)
+		(property "Manufacturer Part Number" "RMCF1206FT10K0"
+			(at 40.64 134.62 0)
+			(hide yes)
+			(show_name no)
+			(do_not_autoplace no)
+			(effects
+				(font
+					(size 1.27 1.27)
+				)
+			)
+		)
+		(property "Vendor Part Number" "RMCF1206FT10K0CT-ND"
+			(at 40.64 134.62 0)
+			(hide yes)
+			(show_name no)
+			(do_not_autoplace no)
+			(effects
+				(font
+					(size 1.27 1.27)
+				)
+			)
+		)
 		(pin "2"
 		)
@@
 			)
 		)
+		(property "Manufacturer Part Number" "RC1206FR-075K1L"
+			(at 367.03 163.83 0)
+			(hide yes)
+			(show_name no)
+			(do_not_autoplace no)
+			(effects
+				(font
+					(size 1.27 1.27)
+				)
+			)
+		)
+		(property "Vendor Part Number" "311-5.10KFRCT-ND"
+			(at 367.03 163.83 0)
+			(hide yes)
+			(show_name no)
+			(do_not_autoplace no)
+			(effects
+				(font
+					(size 1.27 1.27)
+				)
+			)
+		)
 		(pin "2"
 		)
@@
 			)
 		)
+		(property "Manufacturer Part Number" "RC1206FR-0788K7L"
+			(at 184.15 67.31 90)
+			(hide yes)
+			(show_name no)
+			(do_not_autoplace no)
+			(effects
+				(font
+					(size 1.27 1.27)
+				)
+			)
+		)
+		(property "Vendor Part Number" "311-88.7KFRCT-ND"
+			(at 184.15 67.31 90)
+			(hide yes)
+			(show_name no)
+			(do_not_autoplace no)
+			(effects
+				(font
+					(size 1.27 1.27)
+				)
+			)
+		)
 		(pin "2"
 		)
@@
 			)
 		)
+		(property "Manufacturer Part Number" "RMCF1206FT220R"
+			(at 330.2 58.42 90)
+			(hide yes)
+			(show_name no)
+			(do_not_autoplace no)
+			(effects
+				(font
+					(size 1.27 1.27)
+				)
+			)
+		)
+		(property "Vendor Part Number" "RMCF1206FT220RCT-ND"
+			(at 330.2 58.42 90)
+			(hide yes)
+			(show_name no)
+			(do_not_autoplace no)
+			(effects
+				(font
+					(size 1.27 1.27)
+				)
+			)
+		)
 		(pin "2"
 		)
@@
 			)
 		)
+		(property "Manufacturer Part Number" "CRCW120622K1FKEAC"
+			(at 175.26 77.47 0)
+			(hide yes)
+			(show_name no)
+			(do_not_autoplace no)
+			(effects
+				(font
+					(size 1.27 1.27)
+				)
+			)
+		)
+		(property "Vendor Part Number" "541-CRCW120622K1FKEACCT-ND"
+			(at 175.26 77.47 0)
+			(hide yes)
+			(show_name no)
+			(do_not_autoplace no)
+			(effects
+				(font
+					(size 1.27 1.27)
+				)
+			)
+		)
 		(pin "2"
 		)
@@
 			)
 		)
+		(property "Manufacturer Part Number" "RMCF1206FT10K0"
+			(at 378.46 74.93 0)
+			(hide yes)
+			(show_name no)
+			(do_not_autoplace no)
+			(effects
+				(font
+					(size 1.27 1.27)
+				)
+			)
+		)
+		(property "Vendor Part Number" "RMCF1206FT10K0CT-ND"
+			(at 378.46 74.93 0)
+			(hide yes)
+			(show_name no)
+			(do_not_autoplace no)
+			(effects
+				(font
+					(size 1.27 1.27)
+				)
+			)
+		)
 		(pin "2"
 		)
@@
 			)
 		)
+		(property "Manufacturer Part Number" "RMCF1206FT220R"
+			(at 361.95 109.22 0)
+			(hide yes)
+			(show_name no)
+			(do_not_autoplace no)
+			(effects
+				(font
+					(size 1.27 1.27)
+				)
+			)
+		)
+		(property "Vendor Part Number" "RMCF1206FT220RCT-ND"
+			(at 361.95 109.22 0)
+			(hide yes)
+			(show_name no)
+			(do_not_autoplace no)
+			(effects
+				(font
+					(size 1.27 1.27)
+				)
+			)
+		)
 		(pin "2"
 		)
@@
 			)
 		)
+		(property "Manufacturer Part Number" "RC1206FR-075K1L"
+			(at 377.19 163.83 0)
+			(hide yes)
+			(show_name no)
+			(do_not_autoplace no)
+			(effects
+				(font
+					(size 1.27 1.27)
+				)
+			)
+		)
+		(property "Vendor Part Number" "311-5.10KFRCT-ND"
+			(at 377.19 163.83 0)
+			(hide yes)
+			(show_name no)
+			(do_not_autoplace no)
+			(effects
+				(font
+					(size 1.27 1.27)
+				)
+			)
+		)
 		(pin "2"
 		)
@@
 			)
 		)
+		(property "Manufacturer Part Number" "RC1206FR-071KL"
+			(at 394.97 60.96 0)
+			(hide yes)
+			(show_name no)
+			(do_not_autoplace no)
+			(effects
+				(font
+					(size 1.27 1.27)
+				)
+			)
+		)
+		(property "Vendor Part Number" "311-1.00KFRCT-ND"
+			(at 394.97 60.96 0)
+			(hide yes)
+			(show_name no)
+			(do_not_autoplace no)
+			(effects
+				(font
+					(size 1.27 1.27)
+				)
+			)
+		)
 		(pin "2"
 		)
@@
 			(at 332.74 116.84 90)
 			(hide yes)
+			(show_name no)
+			(do_not_autoplace no)
+			(effects
+				(font
+					(size 1.27 1.27)
+				)
+			)
+		)
+		(property "Manufacturer Part Number" "RMCF1206FT220R"
+			(at 332.74 116.84 90)
+			(hide yes)
+			(show_name no)
+			(do_not_autoplace no)
+			(effects
+				(font
+					(size 1.27 1.27)
+				)
+			)
+		)
+		(property "Vendor Part Number" "RMCF1206FT220RCT-ND"
+			(at 332.74 116.84 90)
+			(hide yes)

Commit message: route
Connections:
- net 5V_REGOUT: now reaches C16.1, L1.2, R7.2, U6.1 (VIN), U7.3 (~{CE})
Changed lines of the file:
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@@
+		)
+	)
+	(label "5V_REGOUT"
+		(at 205.74 58.42 0)
+		(effects
+			(font
+				(size 1.27 1.27)
+			)
+			(justify left bottom)
 		)
 	)

Commit message: !!!!!
Connections:
- net ~{ENABLE_1} renamed ENABLE_1
- net ~{ENABLE_2} renamed ENABLE_2
- net ~{ENABLE_3} renamed ENABLE_3
- net ~{ENABLE_4} renamed ENABLE_4
- net ~{ENABLE_5} renamed ENABLE_5
- net ~{ENABLE_6} renamed ENABLE_6
- net ~{ENABLE_7} renamed ENABLE_7
- net ~{ENABLE_8} renamed ENABLE_8
Other:
- sheet Motors & Drivers ports: added ENABLE_[1..8]; removed ~{ENABLE_[1..8]}
Changed lines of the file:
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@@
 		)
 	)
-	(label "~{ENABLE_3}"
+	(label "ENABLE_3"
 		(at 81.28 195.58 0)
 		(effects
@@
 		)
 	)
-	(label "~{ENABLE_1}"
+	(label "ENABLE_1"
 		(at 81.28 190.5 0)
 		(effects
@@
 		)
 	)
-	(label "~{ENABLE_5}"
+	(label "ENABLE_5"
 		(at 81.28 200.66 0)
 		(effects
@@
 		)
 	)
-	(label "~{ENABLE_6}"
+	(label "ENABLE_6"
 		(at 81.28 203.2 0)
 		(effects
@@
 		)
 	)
-	(label "~{ENABLE_8}"
+	(label "ENABLE_8"
 		(at 81.28 208.28 0)
 		(effects
@@
 		)
 	)
-	(label "~{ENABLE_[1..8]}"
+	(label "ENABLE_[1..8]"
 		(at 203.2 166.37 0)
 		(effects
@@
 		)
 	)
-	(label "~{ENABLE_4}"
+	(label "ENABLE_4"
 		(at 81.28 198.12 0)
 		(effects
@@
 		)
 	)
-	(label "~{ENABLE_7}"
+	(label "ENABLE_7"
 		(at 81.28 205.74 0)
 		(effects
@@
 		)
 	)
-	(label "~{ENABLE_2}"
+	(label "ENABLE_2"
 		(at 81.28 193.04 0)
 		(effects
@@
 			)
 		)
-		(pin "~{ENABLE_[1..8]}" output
+		(pin "ENABLE_[1..8]" output
 			(at 218.44 166.37 180)
 			(effects

Commit message: w
Parts:
- added LG1: UCSB_IEEE, footprints:UCSB_IEEE_Logo, symbol symbols:LOGO
- added LG2: UCSB, footprints:UCSB_Medium, symbol symbols:LOGO
Changed lines of the file:
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@@
+	)
+	(symbol
+		(lib_id "symbols:LOGO")
+		(at 279.4 172.72 0)
+		(unit 1)
+		(body_style 1)
+		(exclude_from_sim no)
+		(in_bom no)
+		(on_board yes)
+		(in_pos_files no)
+		(dnp no)
+		(fields_autoplaced yes)
+		(property "Reference" "LG1"
+			(at 283.21 171.4499 0)
+			(show_name no)
+			(do_not_autoplace no)
+			(effects
+				(font
+					(size 1.27 1.27)
+				)
+				(justify left)
+			)
+		)
+		(property "Value" "UCSB_IEEE"
+			(at 283.21 173.9899 0)
+			(show_name no)
+			(do_not_autoplace no)
+			(effects
+				(font
+					(size 1.27 1.27)
+				)
+				(justify left)
+			)
+		)
+		(property "Footprint" "footprints:UCSB_IEEE_Logo"
+			(at 279.4 172.72 0)
+			(hide yes)
+			(show_name no)
+			(do_not_autoplace no)
+			(effects
+				(font
+					(size 1.27 1.27)
+				)
+			)
+		)
+		(property "Datasheet" ""
+			(at 279.4 172.72 0)
+			(hide yes)
+			(show_name no)
+			(do_not_autoplace no)
+			(effects
+				(font
+					(size 1.27 1.27)
+				)
+			)
+		)
+		(property "Description" ""
+			(at 279.4 172.72 0)
+			(hide yes)
+			(show_name no)
+			(do_not_autoplace no)
+			(effects
+				(font
+					(size 1.27 1.27)
+				)
+			)
+		)
+		(instances
+			(project "stepper_music"
+				(path "/c1f09015-b8de-4a7b-b4da-e4fcb6b13235"
+					(reference "LG1")
+					(unit 1)
+				)
+			)
+		)
 	)
 	(symbol
@@
 					(unit 1)
 				)
+			)
+		)
+	)
+	(symbol
+		(lib_id "symbols:LOGO")
+		(at 279.4 177.8 0)
+		(unit 1)
+		(body_style 1)
+		(exclude_from_sim no)
+		(in_bom no)
+		(on_board yes)
+		(in_pos_files no)
+		(dnp no)
+		(fields_autoplaced yes)
+		(property "Reference" "LG2"
+			(at 283.21 176.5299 0)
+			(show_name no)
+			(do_not_autoplace no)
+			(effects
+				(font
+					(size 1.27 1.27)
+				)
+				(justify left)
+			)
+		)
+		(property "Value" "UCSB"
+			(at 283.21 179.0699 0)
+			(show_name no)
+			(do_not_autoplace no)
+			(effects
+				(font
+					(size 1.27 1.27)
+				)
+				(justify left)
+			)
+		)
+		(property "Footprint" "footprints:UCSB_Medium"
+			(at 279.4 177.8 0)
+			(hide yes)
+			(show_name no)
+			(do_not_autoplace no)
+			(effects
+				(font
+					(size 1.27 1.27)
+				)
+			)
+		)
+		(property "Datasheet" ""
+			(at 279.4 177.8 0)
+			(hide yes)
+			(show_name no)
+			(do_not_autoplace no)
+			(effects
+				(font
+					(size 1.27 1.27)
+				)
+			)
+		)
+		(property "Description" ""
+			(at 279.4 177.8 0)
+			(hide yes)
+			(show_name no)
+			(do_not_autoplace no)
+			(effects
+				(font
+					(size 1.27 1.27)
+				)
+			)
+		)
+		(instances
+			(project "stepper_music"
+				(path "/c1f09015-b8de-4a7b-b4da-e4fcb6b13235"
+					(reference "LG2")
+					(unit 1)
+				)

Commit message: holes
Parts:
- added H1, H2, H3, H4: Hole, MountingHole:MountingHole_3.2mm_M3_DIN965, symbol Mechanical:MountingHole

Commit message: w
Parts:
- J5: footprint Connector_AMASS:AMASS_XT30PW-M_1x02_P2.50mm_Horizontal -> Connector_AMASS:AMASS_XT60PW-M_1x02_P7.20mm_Horizontal; Manufacturer Part Number XT30PW-M30 -> XT60PW-M30; Vendor Part Number 2844399 -> 2844439
Changed lines of the file:
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@@
 			)
 		)
-		(property "Footprint" "Connector_AMASS:AMASS_XT30PW-M_1x02_P2.50mm_Horizontal"
+		(property "Footprint" "Connector_AMASS:AMASS_XT60PW-M_1x02_P7.20mm_Horizontal"
 			(at 29.21 58.42 0)
 			(hide yes)
@@
 			)
 		)
-		(property "Manufacturer Part Number" "XT30PW-M30"
+		(property "Manufacturer Part Number" "XT60PW-M30"
 			(at 29.21 58.42 0)
 			(hide yes)
@@
 			)
 		)
-		(property "Vendor Part Number" "2844399"
+		(property "Vendor Part Number" "2844439"
 			(at 29.21 58.42 0)
 			(hide yes)
