File: pcb/1.0/driver.kicad_sch (KiCad schematic)
At the start: 14 parts, among them U8 A4988SETTR-T

Commit message: fixes
Parts:
- removed HS1: Heatsink, symbol Mechanical:Heatsink
Changed lines of the file:
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@@
-	)
-	(symbol
-		(lib_id "Mechanical:Heatsink")
-		(at 127 63.5 0)
-		(unit 1)
-		(body_style 1)
-		(exclude_from_sim no)
-		(in_bom yes)
-		(on_board no)
-		(in_pos_files no)
-		(dnp no)
-		(fields_autoplaced yes)
-		(property "Reference" "HS1"
-			(at 130.81 60.3249 0)
-			(show_name no)
-			(do_not_autoplace no)
-			(effects
-				(font
-					(size 1.27 1.27)
-				)
-				(justify left)
-			)
-		)
-		(property "Value" "Heatsink"
-			(at 130.81 62.8649 0)
-			(show_name no)
-			(do_not_autoplace no)
-			(effects
-				(font
-					(size 1.27 1.27)
-				)
-				(justify left)
-			)
-		)
-		(property "Footprint" ""
-			(at 127.3048 63.5 0)
-			(hide yes)
-			(show_name no)
-			(do_not_autoplace no)
-			(effects
-				(font
-					(size 1.27 1.27)
-				)
-			)
-		)
-		(property "Datasheet" ""
-			(at 127.3048 63.5 0)
-			(hide yes)
-			(show_name no)
-			(do_not_autoplace no)
-			(effects
-				(font
-					(size 1.27 1.27)
-				)
-			)
-		)
-		(property "Description" "Heatsink"
-			(at 127 63.5 0)
-			(hide yes)
-			(show_name no)
-			(do_not_autoplace no)
-			(effects
-				(font
-					(size 1.27 1.27)
-				)
-			)
-		)
-		(instances
-			(project "stepper_music"
-				(path "/c1f09015-b8de-4a7b-b4da-e4fcb6b13235/65bd6e05-ecc8-4355-bcb4-1d1e2a69c8df/08eedecc-4324-421b-8619-41688fa76849"
-					(reference "HS2")
-					(unit 1)
-				)
-				(path "/c1f09015-b8de-4a7b-b4da-e4fcb6b13235/65bd6e05-ecc8-4355-bcb4-1d1e2a69c8df/5bbe4836-44e8-4f24-b1ae-ed92f44e542e"
-					(reference "HS8")
-					(unit 1)
-				)
-				(path "/c1f09015-b8de-4a7b-b4da-e4fcb6b13235/65bd6e05-ecc8-4355-bcb4-1d1e2a69c8df/60dae45a-bf18-4832-b54f-8416f293d78e"
-					(reference "HS6")
-					(unit 1)
-				)
-				(path "/c1f09015-b8de-4a7b-b4da-e4fcb6b13235/65bd6e05-ecc8-4355-bcb4-1d1e2a69c8df/627db15f-8545-460a-83cc-41b559e00082"
-					(reference "HS4")
-					(unit 1)
-				)
-				(path "/c1f09015-b8de-4a7b-b4da-e4fcb6b13235/65bd6e05-ecc8-4355-bcb4-1d1e2a69c8df/7c709d1e-4f00-4901-a1f8-f6836429dc30"
-					(reference "HS5")
-					(unit 1)
-				)
-				(path "/c1f09015-b8de-4a7b-b4da-e4fcb6b13235/65bd6e05-ecc8-4355-bcb4-1d1e2a69c8df/d586785d-5219-4549-8fd2-ceb2e303be2c"
-					(reference "HS1")
-					(unit 1)
-				)
-				(path "/c1f09015-b8de-4a7b-b4da-e4fcb6b13235/65bd6e05-ecc8-4355-bcb4-1d1e2a69c8df/f069a111-c28e-40fd-84d8-8b318c4858de"
-					(reference "HS7")
-					(unit 1)
-				)
-				(path "/c1f09015-b8de-4a7b-b4da-e4fcb6b13235/65bd6e05-ecc8-4355-bcb4-1d1e2a69c8df/f7e37d7f-d74d-464d-bb2e-26fef4e38440"
-					(reference "HS3")
-					(unit 1)
-				)
-			)
-		)
 	)
 	(symbol
