File: pcb/1.0/stepper_music.kicad_pcb (KiCad board)
At the start: 4 copper layers, 75 x 155 mm, 168 parts, among them J1 USB_C_Receptacle, J2 Conn_ST_STDC14, J3 MIDI IN, J4 MIDI THRU, J5 Conn_01x02, M1 Stepper_Motor_unipolar_6pin, M2 Stepper_Motor_unipolar_6pin, M3 Stepper_Motor_unipolar_6pin, M4 Stepper_Motor_unipolar_6pin, M5 Stepper_Motor_unipolar_6pin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

Commit message: fixes
Parts:
- R7: value 0Ω -> 88.7kΩ
- moved J1 3.00 mm to (61.0, 158.0)
- moved R1 3.00 mm to (62.5, 164.8)
- moved R2 3.00 mm to (62.5, 151.2)
Routing:
- net /USB_D+: track 28.1 -> 22.1 mm
- net /USB_D-: track 21.9 -> 18.9 mm
- net /VBUS: track 66.6 -> 63.6 mm
