File: pcb/1.0/stepper_music.kicad_sch (KiCad schematic)
At the start: 56 parts, among them J1 USB_C_Receptacle, J2 Conn_ST_STDC14, J3 MIDI IN, J4 MIDI THRU, J5 Conn_01x02, U1 STM32F401RCTx, U2 6N138, U3 LD1117S33TR_SOT223, U4 LMR50410, U5 SN74LV1T34DBV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

Commit message: fixes
Parts:
- R7: value 0Ω -> 88.7kΩ; Manufacturer Part Number (none) -> RC1206FR-0788K7L; Vendor Part Number (none) -> 311-88.7KFRCT-ND
- R8: now fitted
Changed lines of the file:
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@@
 			)
 		)
-		(property "Value" "0Ω"
+		(property "Value" "88.7kΩ"
 			(at 184.15 63.5 90)
 			(show_name no)
@@
 			)
 		)
-		(property "Manufacturer Part Number" ""
+		(property "Manufacturer Part Number" "RC1206FR-0788K7L"
 			(at 184.15 67.31 90)
 			(hide yes)
@@
 			)
 		)
-		(property "Vendor Part Number" ""
+		(property "Vendor Part Number" "311-88.7KFRCT-ND"
 			(at 184.15 67.31 90)
 			(hide yes)
@@
 		(on_board yes)
 		(in_pos_files yes)
-		(dnp yes)
+		(dnp no)
 		(fields_autoplaced yes)
 		(property "Reference" "R8"
